File: retro-ciaa.sch (KiCad schematic (older format))
At the start: 113 parts, among them P1 VIDEO OUT, P10 SPI PORT, P11 I²C PORT, P12 ADC PORT, P2 RGBHV TEST POINTS, P3 GAMEPAD 2, P4 P2 PORT, P5 P1 PORT, P6 GAMEPAD 1, P7 WIFI MODULE UART, P8 WIFI MODULE BOOT, P9 AUDIO LINE OUT, U1 VGA SYNC/JOY BUFFER, U2 VGA RGB BUFFER, U3 E-DDC I²C BUFFER, U4 1Mbit EEPROM, U5 I²S AUDIO DAC, U6 WIFI MODULE, U7 BACKLIGHT COVER

Commit message: Esquematico A3 terminado
Parts:
- P4: symbol EDU-CIAA_P2 -> EDU-CIAA_P2_2
- P5: symbol EDU-CIAA_P1 -> EDU-CIAA_P1_2
- U1, U2: symbol SN74ALVC245 -> SN74ALVC245-RESCUE-retro-ciaa
- U5: symbol PCM5100A -> PCM5100A-RESCUE-retro-ciaa
- U6: symbol ESP-WROOM-32 -> ESP-WROOM-32-RESCUE-retro-ciaa
Connections:
- wire segments 283 -> 317
Other:
- moved on the sheet: C20, P10, P11, P12, P7, P8, R34, R35, R41, U4
