File: storage.sch (KiCad schematic (older format))
At the start: 3 parts, among them U4 1Mbit EEPROM

Commit message: Cambios menores
Connections:
- net +3V3: now also U4.8 (VCC); no longer U4.6 (SCL)
- net GND: now also U4.4 (VSS), U4.7 (~WC); no longer U4.1 (DU), U4.5 (SDA)
- net [SCL]: now also U4.6 (SCL); no longer U4.7 (~WC)
- net [SDA]: now also U4.5 (SDA); no longer U4.4 (VSS)
Other:
- note added: "Decoupling capacitors. \nPlace as close as possible to the affected IC pin."
Changed lines of the file:
@@
 	1    0    0    -1
 $EndComp
-Text Label 6300 3000 0    60   ~ 0
-GND
-NoConn ~ 5300 2900
-Text Label 5300 3200 2    60   ~ 0
-GND
 Text Notes 5500 3850 0    60   ~ 0
 R/W 101011X
@@
 Text Label 5200 4400 0    60   ~ 0
 EEPROM_VCC
-Text Label 6300 2900 0    60   ~ 0
+Text Label 5300 2900 2    60   ~ 0
 EEPROM_VCC
 Wire Wire Line
@@
 	5900 4400 5900 4500
 Connection ~ 5900 4400
-Text HLabel 7000 3100 2    60   Input ~ 0
+Text HLabel 7000 2900 2    60   Input ~ 0
 [SCL]
-Text HLabel 7000 3200 2    60   BiDi ~ 0
+Text HLabel 7000 3000 2    60   BiDi ~ 0
 [SDA]
 Wire Wire Line
-	6300 3100 7000 3100
+	6300 2900 7000 2900
 Wire Wire Line
-	7000 3200 6300 3200
+	7000 3000 6300 3000
 Text Label 6300 7500 2    60   ~ 0
 3V3
@@
 Wire Wire Line
 	6700 7300 6700 7400
+Text Notes 5200 5200 0    60   ~ 0
+Decoupling capacitors. \nPlace as close as possible to the affected IC pin.
+NoConn ~ 5300 3200
+$Comp
+L GND #PWR083
+U 1 1 5BCAEF3C
+P 6400 3400
+F 0 "#PWR083" H 6400 3150 50  0001 C CNN
+F 1 "GND" H 6400 3250 50  0000 C CNN
+F 2 "" H 6400 3400 50  0000 C CNN
+F 3 "" H 6400 3400 50  0000 C CNN
+	1    6400 3400
+	1    0    0    -1
+$EndComp
+Wire Wire Line
+	6300 3100 6400 3100
+Wire Wire Line
+	6400 3100 6400 3400
+Wire Wire Line
+	6300 3200 6400 3200
+Connection ~ 6400 3200
 $EndSCHEMATC

Commit message: Limpieza de etiquetas de alimentacion
Changed lines of the file:
@@
 $EndComp
 $Comp
-L +3.3V #PWR079
+L +3.3V #PWR073
 U 1 1 5BD57DA9
 P 6400 4400
-F 0 "#PWR079" H 6400 4250 50  0001 C CNN
+F 0 "#PWR073" H 6400 4250 50  0001 C CNN
 F 1 "+3.3V" H 6400 4540 50  0000 C CNN
 F 2 "" H 6400 4400 50  0000 C CNN
@@
 $EndComp
 $Comp
-L GND #PWR080
+L GND #PWR074
 U 1 1 5BD57DAF
 P 6400 4900
-F 0 "#PWR080" H 6400 4650 50  0001 C CNN
+F 0 "#PWR074" H 6400 4650 50  0001 C CNN
 F 1 "GND" H 6400 4750 50  0000 C CNN
 F 2 "" H 6400 4900 50  0000 C CNN
@@
 Wire Wire Line
 	7000 3000 6300 3000
-Text Label 6300 7500 2    60   ~ 0
+Text Label 6700 7500 2    60   ~ 0
 3V3
 $Comp
-L +3.3V #PWR081
+L +3.3V #PWR075
 U 1 1 5BD60C63
-P 6100 7400
-F 0 "#PWR081" H 6100 7250 50  0001 C CNN
-F 1 "+3.3V" H 6100 7540 50  0000 C CNN
-F 2 "" H 6100 7400 50  0000 C CNN
-F 3 "" H 6100 7400 50  0000 C CNN
-	1    6100 7400
+P 6500 7400
+F 0 "#PWR075" H 6500 7250 50  0001 C CNN
+F 1 "+3.3V" H 6500 7540 50  0000 C CNN
+F 2 "" H 6500 7400 50  0000 C CNN
+F 3 "" H 6500 7400 50  0000 C CNN
+	1    6500 7400
 	1    0    0    -1
 $EndComp
-$Comp
-L GND #PWR082
-U 1 1 5BD60C69
-P 6700 7400
-F 0 "#PWR082" H 6700 7150 50  0001 C CNN
-F 1 "GND" H 6700 7250 50  0000 C CNN
-F 2 "" H 6700 7400 50  0000 C CNN
-F 3 "" H 6700 7400 50  0000 C CNN
-	1    6700 7400
-	1    0    0    -1
-$EndComp
-Text Label 6500 7300 0    60   ~ 0
-GND
 Wire Wire Line
-	6100 7400 6100 7500
+	6500 7400 6500 7500
 Wire Wire Line
-	6100 7500 6300 7500
-Wire Wire Line
-	6500 7300 6700 7300
-Wire Wire Line
-	6700 7300 6700 7400
+	6500 7500 6700 7500
 Text Notes 5200 5200 0    60   ~ 0
 Decoupling capacitors. \nPlace as close as possible to the affected IC pin.
 NoConn ~ 5300 3200
 $Comp
-L GND #PWR083
+L GND #PWR076
 U 1 1 5BCAEF3C
 P 6400 3400
-F 0 "#PWR083" H 6400 3150 50  0001 C CNN
+F 0 "#PWR076" H 6400 3150 50  0001 C CNN
 F 1 "GND" H 6400 3250 50  0000 C CNN
 F 2 "" H 6400 3400 50  0000 C CNN
