File: wifi.sch (KiCad schematic (older format))
At the start: 7 parts, among them P7 WIFI MODULE UART, P8 WIFI MODULE BOOT, U6 WIFI MODULE

Commit message: Cambios menores
Other:
- note added: "Decoupling capacitors. \nPlace as close as possible to the affected IC pin."
Changed lines of the file:
@@
 WM_3V3
 $Comp
-L +3.3V #PWR052
+L +3.3V #PWR049
 U 1 1 5BD1D8EA
 P 5100 2600
-F 0 "#PWR052" H 5100 2450 50  0001 C CNN
+F 0 "#PWR049" H 5100 2450 50  0001 C CNN
 F 1 "+3.3V" H 5100 2740 50  0000 C CNN
 F 2 "" H 5100 2600 50  0000 C CNN
@@
 Connection ~ 5100 3100
 $Comp
-L GND #PWR053
+L GND #PWR050
 U 1 1 5BD1D8F6
 P 5100 3500
-F 0 "#PWR053" H 5100 3250 50  0001 C CNN
+F 0 "#PWR050" H 5100 3250 50  0001 C CNN
 F 1 "GND" H 5100 3350 50  0000 C CNN
 F 2 "" H 5100 3500 50  0000 C CNN
@@
 	-1   0    0    1
 $EndComp
-Text Notes 5400 2750 0    60   ~ 0
+Text Notes 5700 3500 0    60   ~ 0
 Required RC\ndelay circuit
 $Comp
@@
 WM_AT_TXD
 $Comp
-L GND #PWR054
+L GND #PWR051
 U 1 1 5BD1D936
 P 4500 5100
-F 0 "#PWR054" H 4500 4850 50  0001 C CNN
+F 0 "#PWR051" H 4500 4850 50  0001 C CNN
 F 1 "GND" H 4500 4950 50  0000 C CNN
 F 2 "" H 4500 5100 50  0000 C CNN
@@
 WM_3V3
 $Comp
-L +3.3V #PWR055
+L +3.3V #PWR052
 U 1 1 5BD22609
 P 9100 1600
-F 0 "#PWR055" H 9100 1450 50  0001 C CNN
+F 0 "#PWR052" H 9100 1450 50  0001 C CNN
 F 1 "+3.3V" H 9100 1740 50  0000 C CNN
 F 2 "" H 9100 1600 50  0000 C CNN
@@
 $EndComp
 $Comp
-L GND #PWR056
+L GND #PWR053
 U 1 1 5BD2260F
 P 9100 2100
-F 0 "#PWR056" H 9100 1850 50  0001 C CNN
+F 0 "#PWR053" H 9100 1850 50  0001 C CNN
 F 1 "GND" H 9100 1950 50  0000 C CNN
 F 2 "" H 9100 2100 50  0000 C CNN
@@
 3V3
 $Comp
-L +3.3V #PWR057
+L +3.3V #PWR054
 U 1 1 5BD5E07B
 P 6100 7400
-F 0 "#PWR057" H 6100 7250 50  0001 C CNN
+F 0 "#PWR054" H 6100 7250 50  0001 C CNN
 F 1 "+3.3V" H 6100 7540 50  0000 C CNN
 F 2 "" H 6100 7400 50  0000 C CNN
@@
 $EndComp
 $Comp
-L GND #PWR058
+L GND #PWR055
 U 1 1 5BD5E081
 P 6700 7400
-F 0 "#PWR058" H 6700 7150 50  0001 C CNN
+F 0 "#PWR055" H 6700 7150 50  0001 C CNN
 F 1 "GND" H 6700 7250 50  0000 C CNN
 F 2 "" H 6700 7400 50  0000 C CNN
@@
 Wire Wire Line
 	6700 7300 6700 7400
+Text Notes 7900 2400 0    60   ~ 0
+Decoupling capacitors. \nPlace as close as possible to the affected IC pin.
 $EndSCHEMATC

Commit message: Nuevo layout, mejoras y modificaciones del revisor
Parts:
- U6: symbol ESP-WROOM-32-RESCUE-retro-ciaa -> ESP-WROOM-32
Other:
- moved on the sheet: C16, R36
Changed lines of the file:
@@
 LIBS:contrib
 LIBS:valves
-LIBS:salmon
+LIBS:retro-ciaa
 LIBS:retro-ciaa-cache
 EELAYER 25 0
@@
 encoding utf-8
 Sheet 5 8
-Title "RETRO-CIAA / WI-FI & BLUETOOTH"
-Date "2018-10-19"
+Title "WI-FI & BLUETOOTH"
+Date "2018-10-20"
 Rev "1.1.1"
-Comp "Salmon Robotics"
+Comp "http://www.retro-ciaa.com"
 Comment1 "All resistors 1% & 0603\" unless otherwise noted"
 Comment2 "ERC check OK on 2018-10-19"
@@
 $EndDescr
 $Comp
-L ESP-WROOM-32-RESCUE-retro-ciaa U6
+L ESP-WROOM-32 U6
 U 1 1 5BD1D8D1
 P 3600 4000
@@
 L +3.3V #PWR049
 U 1 1 5BD1D8EA
-P 5100 2600
-F 0 "#PWR049" H 5100 2450 50  0001 C CNN
-F 1 "+3.3V" H 5100 2740 50  0000 C CNN
-F 2 "" H 5100 2600 50  0000 C CNN
-F 3 "" H 5100 2600 50  0000 C CNN
-	1    5100 2600
-	1    0    0    -1
-$EndComp
-Wire Wire Line
-	5100 2700 5100 2600
-Wire Wire Line
-	4400 3100 5800 3100
-Wire Wire Line
-	5100 3000 5100 3200
-Connection ~ 5100 3100
+P 5400 2600
+F 0 "#PWR049" H 5400 2450 50  0001 C CNN
+F 1 "+3.3V" H 5400 2740 50  0000 C CNN
+F 2 "" H 5400 2600 50  0000 C CNN
+F 3 "" H 5400 2600 50  0000 C CNN
+	1    5400 2600
+	1    0    0    -1
+$EndComp
+Wire Wire Line
+	5400 2700 5400 2600
+Wire Wire Line
+	4400 3100 6100 3100
+Wire Wire Line
+	5400 3000 5400 3200
+Connection ~ 5400 3100
 $Comp
 L GND #PWR050
 U 1 1 5BD1D8F6
-P 5100 3500
-F 0 "#PWR050" H 5100 3250 50  0001 C CNN
-F 1 "GND" H 5100 3350 50  0000 C CNN
-F 2 "" H 5100 3500 50  0000 C CNN
-F 3 "" H 5100 3500 50  0000 C CNN
-	1    5100 3500
+P 5400 3600
+F 0 "#PWR050" H 5400 3350 50  0001 C CNN
+F 1 "GND" H 5400 3450 50  0000 C CNN
+F 2 "" H 5400 3600 50  0000 C CNN
+F 3 "" H 5400 3600 50  0000 C CNN
+	1    5400 3600
 	1    0    0    -1
 $EndComp
@@
 L C C16
 U 1 1 5BD1D908
-P 5100 3350
-F 0 "C16" H 4900 3250 50  0000 L CNN
-F 1 "100nF" H 4750 3350 50  0000 L CNN
-F 2 "Capacitors_SMD:C_0603" H 5100 3350 31  0001 C CNN
-F 3 "885012206071" H 4900 3450 31  0000 C CNN
-	1    5100 3350
+P 5400 3350
+F 0 "C16" H 5200 3250 50  0000 L CNN
+F 1 "100nF" H 5050 3350 50  0000 L CNN
+F 2 "Capacitors_SMD:C_0603" H 5400 3350 31  0001 C CNN
+F 3 "885012206071" H 5200 3450 31  0000 C CNN
+	1    5400 3350
 	-1   0    0    1
 $EndComp
-Text Notes 5700 3500 0    60   ~ 0
+Text Notes 5600 3800 0    60   ~ 0
 Required RC\ndelay circuit
 $Comp
 L R R36
 U 1 1 5BD1D910
-P 5100 2850
-F 0 "R36" V 5000 2850 50  0000 C CNN
-F 1 "10K" V 5100 2850 50  0000 C CNN
-F 2 "Resistors_SMD:R_0603" V 5030 2850 31  0001 C CNN
-F 3 "RC0603FR-0710KL" V 5200 2850 31  0000 C CNN
-	1    5100 2850
+P 5400 2850
+F 0 "R36" V 5300 2850 50  0000 C CNN
+F 1 "10K" V 5400 2850 50  0000 C CNN
+F 2 "Resistors_SMD:R_0603" V 5330 2850 31  0001 C CNN
+F 3 "RC0603FR-0710KL" V 5500 2850 31  0000 C CNN
+	1    5400 2850
 	1    0    0    -1
 $EndComp
@@
 Text HLabel 2100 3800 0    60   Input ~ 0
 [WM_AT_TXD]
-Text HLabel 5800 3100 2    60   Input ~ 0
+Text HLabel 6100 3100 2    60   Input ~ 0
 [WM_EN]
 Wire Wire Line
@@
 Text Notes 7900 2400 0    60   ~ 0
 Decoupling capacitors. \nPlace as close as possible to the affected IC pin.
+Wire Wire Line
+	5400 3600 5400 3500
 $EndSCHEMATC

Commit message: Limpieza de etiquetas de alimentacion
Changed lines of the file:
@@
 WM_3V3
 $Comp
-L +3.3V #PWR049
+L +3.3V #PWR045
 U 1 1 5BD1D8EA
 P 5400 2600
-F 0 "#PWR049" H 5400 2450 50  0001 C CNN
+F 0 "#PWR045" H 5400 2450 50  0001 C CNN
 F 1 "+3.3V" H 5400 2740 50  0000 C CNN
 F 2 "" H 5400 2600 50  0000 C CNN
@@
 Connection ~ 5400 3100
 $Comp
-L GND #PWR050
+L GND #PWR046
 U 1 1 5BD1D8F6
 P 5400 3600
-F 0 "#PWR050" H 5400 3350 50  0001 C CNN
+F 0 "#PWR046" H 5400 3350 50  0001 C CNN
 F 1 "GND" H 5400 3450 50  0000 C CNN
 F 2 "" H 5400 3600 50  0000 C CNN
@@
 WM_AT_TXD
 $Comp
-L GND #PWR051
+L GND #PWR047
 U 1 1 5BD1D936
 P 4500 5100
-F 0 "#PWR051" H 4500 4850 50  0001 C CNN
+F 0 "#PWR047" H 4500 4850 50  0001 C CNN
 F 1 "GND" H 4500 4950 50  0000 C CNN
 F 2 "" H 4500 5100 50  0000 C CNN
@@
 WM_3V3
 $Comp
-L +3.3V #PWR052
+L +3.3V #PWR048
 U 1 1 5BD22609
 P 9100 1600
-F 0 "#PWR052" H 9100 1450 50  0001 C CNN
+F 0 "#PWR048" H 9100 1450 50  0001 C CNN
 F 1 "+3.3V" H 9100 1740 50  0000 C CNN
 F 2 "" H 9100 1600 50  0000 C CNN
@@
 $EndComp
 $Comp
-L GND #PWR053
+L GND #PWR049
 U 1 1 5BD2260F
 P 9100 2100
-F 0 "#PWR053" H 9100 1850 50  0001 C CNN
+F 0 "#PWR049" H 9100 1850 50  0001 C CNN
 F 1 "GND" H 9100 1950 50  0000 C CNN
 F 2 "" H 9100 2100 50  0000 C CNN
@@
 Wire Wire Line
 	2800 3800 2100 3800
-Text Label 6300 7500 2    60   ~ 0
-3V3
-$Comp
-L +3.3V #PWR054
-U 1 1 5BD5E07B
-P 6100 7400
-F 0 "#PWR054" H 6100 7250 50  0001 C CNN
-F 1 "+3.3V" H 6100 7540 50  0000 C CNN
-F 2 "" H 6100 7400 50  0000 C CNN
-F 3 "" H 6100 7400 50  0000 C CNN
-	1    6100 7400
-	1    0    0    -1
-$EndComp
-$Comp
-L GND #PWR055
+$Comp
+L GND #PWR050
 U 1 1 5BD5E081
 P 6700 7400
-F 0 "#PWR055" H 6700 7150 50  0001 C CNN
+F 0 "#PWR050" H 6700 7150 50  0001 C CNN
 F 1 "GND" H 6700 7250 50  0000 C CNN
 F 2 "" H 6700 7400 50  0000 C CNN
@@
 GND
 Wire Wire Line
-	6100 7400 6100 7500
-Wire Wire Line
-	6100 7500 6300 7500
-Wire Wire Line
 	6500 7300 6700 7300
